File: PCB V2.1/Power_system.sch (KiCad schematic (older format))
At the start: 18 parts, among them J3 B2B-PH-K-S(LF)(SN), J4 B3B-PH-K-S(LF)(SN), Q1 DMG2307L-7, Q2 DMG2307L-7, U2 BQ24210DQCT, U3 AZ1117CR-3.3TRG1_1

Commit message: App Notes
App notes added to datasheets folder.
Connections:
- wire segments 55 -> 41
Changed lines of the file:
@@
 $EndComp
 Wire Wire Line
-	800  2575 2200 2575
-Wire Wire Line
-	2200 2575 7500 2575
-Wire Wire Line
-	7500 2575 7775 2575
-Wire Wire Line
-	2200 2575 2200 2900
-Wire Wire Line
-	2200 2900 2200 3400
-Wire Wire Line
-	2200 2900 3500 2900
-Wire Wire Line
-	3500 2900 4100 2900
-Wire Wire Line
-	4100 2900 4675 2900
-Wire Wire Line
-	5775 2900 6900 2900
-Wire Wire Line
-	6900 2900 7100 2900
-Wire Wire Line
-	7100 2900 7275 2900
-Wire Wire Line
-	7275 2900 7675 2900
+	800  2575 7775 2575
+Wire Wire Line
+	2200 2575 2200 3400
+Wire Wire Line
+	2200 2900 4675 2900
+Wire Wire Line
+	5775 2900 7675 2900
 Wire Wire Line
 	8275 2575 8275 2900
@@
 Connection ~ 7500 2575
 Wire Wire Line
-	8275 2900 8900 2900
-Wire Wire Line
-	8900 2900 9100 2900
-Wire Wire Line
-	10100 2900 10325 2900
-Wire Wire Line
-	10325 2900 10875 2900
+	8275 2900 9100 2900
+Wire Wire Line
+	10100 2900 10875 2900
 Connection ~ 10325 2900
 $Comp
-L +3.3V #PWR38
+L +3.3V #PWR033
 U 1 1 57D80E79
 P 10875 2900
-F 0 "#PWR38" H 10875 2750 50  0001 C CNN
+F 0 "#PWR033" H 10875 2750 50  0001 C CNN
 F 1 "+3.3V" H 10875 3040 50  0000 C CNN
 F 2 "" H 10875 2900 50  0000 C CNN
@@
 $EndComp
 $Comp
-L GND #PWR37
+L GND #PWR034
 U 1 1 57D80F19
 P 9600 3350
-F 0 "#PWR37" H 9600 3100 50  0001 C CNN
+F 0 "#PWR034" H 9600 3100 50  0001 C CNN
 F 1 "GND" H 9600 3200 50  0000 C CNN
 F 2 "" H 9600 3350 50  0000 C CNN
@@
 $EndComp
 Wire Wire Line
-	8900 3350 9600 3350
-Wire Wire Line
-	9600 3350 10325 3350
+	8900 3350 10325 3350
 Connection ~ 9600 3350
 Connection ~ 8900 2900
@@
 	5775 3200 6000 3200
 Wire Wire Line
-	6000 3200 6000 3325
-Wire Wire Line
-	6000 3325 6000 4875
+	6000 3200 6000 4875
 Wire Wire Line
 	6000 4875 4675 4875
@@
 Connection ~ 6000 3325
 $Comp
-L GND #PWR35
+L GND #PWR035
 U 1 1 57D82F5E
 P 5225 4600
-F 0 "#PWR35" H 5225 4350 50  0001 C CNN
+F 0 "#PWR035" H 5225 4350 50  0001 C CNN
 F 1 "GND" H 5225 4450 50  0000 C CNN
 F 2 "" H 5225 4600 50  0000 C CNN
@@
 	5225 4000 5225 4600
 Wire Wire Line
-	5125 4600 5225 4600
-Wire Wire Line
-	5225 4600 5325 4600
+	5125 4600 5325 4600
 Wire Wire Line
 	5325 4600 5325 4000
@@
 $EndComp
 $Comp
-L GND #PWR34
+L GND #PWR036
 U 1 1 57D853F5
 P 4100 3350
-F 0 "#PWR34" H 4100 3100 50  0001 C CNN
+F 0 "#PWR036" H 4100 3100 50  0001 C CNN
 F 1 "GND" H 4100 3200 50  0000 C CNN
 F 2 "" H 4100 3350 50  0000 C CNN
@@
 $EndComp
 $Comp
-L GND #PWR33
+L GND #PWR037
 U 1 1 57D89874
 P 2750 3625
-F 0 "#PWR33" H 2750 3375 50  0001 C CNN
+F 0 "#PWR037" H 2750 3375 50  0001 C CNN
 F 1 "GND" H 2750 3475 50  0000 C CNN
 F 2 "" H 2750 3625 50  0000 C CNN
@@
 Connection ~ 2200 2900
 $Comp
-L GND #PWR32
+L GND #PWR038
 U 1 1 57D8ABE6
 P 2725 4125
-F 0 "#PWR32" H 2725 3875 50  0001 C CNN
+F 0 "#PWR038" H 2725 3875 50  0001 C CNN
 F 1 "GND" H 2725 3975 50  0000 C CNN
 F 2 "" H 2725 4125 50  0000 C CNN
@@
 $EndComp
 $Comp
-L GND #PWR36
+L GND #PWR039
 U 1 1 57E05471
 P 8775 4525
-F 0 "#PWR36" H 8775 4275 50  0001 C CNN
+F 0 "#PWR039" H 8775 4275 50  0001 C CNN
 F 1 "GND" H 8775 4375 50  0000 C CNN
 F 2 "" H 8775 4525 50  0000 C CNN
@@
 	8775 4225 8775 4525
 Wire Wire Line
-	8175 4225 8100 4225
-Wire Wire Line
-	8100 4225 7975 4225
+	7975 4225 8175 4225
 Wire Wire Line
 	8100 4225 8100 5200
