File: PCB V2.1/SunLeaf_V2.kicad_pcb (KiCad board)
At the start: 4 copper layers, 77.5 x 40 mm, 155 parts, among them IC1 ESP_09, J1 20021121-00010C4LF, J10 B4B-PH-K-S(LF)(SN), J11 B4B-PH-K-S(LF)(SN), J12 B4B-PH-K-S(LF)(SN), J13 B4B-PH-K-S(LF)(SN), J14 B4B-PH-K-S(LF)(SN), J15 B4B-PH-K-S(LF)(SN), J16 B4B-PH-K-S(LF)(SN), J2 0475890001-MicroUSBPort, J3 B2B-PH-K-S(LF)(SN), J4 B3B-PH-K-S(LF)(SN), J5 B4B-PH-K-S(LF)(SN), J6 B4B-PH-K-S(LF)(SN), J7 B4B-PH-K-S(LF)(SN), J8 B4B-PH-K-S(LF)(SN), J9 B4B-PH-K-S(LF)(SN), P2 CONN_01X03, Q1 DMG2307L-7, Q2 DMG2307L-7, SW1 B3U-1000P, SW2 B3U-1000P, T1 1909763-1, U1 STM32F446RET6_-_TQFP64, U2 BQ24210DQCT, U3 AZ1117CR-3.3TRG1_1, U4 74HC4052D, U5 PCA9518DBQR, X1 ABM3B8.000MHZB2T, X2 ABS07-32.768KHZ-9-T

Commit message: Images
Images added and organized
Parts:
- added TP35: TEST_POINT, PCB_Footprints:TEST_POINT, F.Cu at (51.0, 68.4)
- added TP36: TEST_POINT, PCB_Footprints:TEST_POINT, F.Cu at (54.9, 68.5)
- moved FD2 4.95 mm to (57.3, 68.7)
Routing:
- net GND: track 256.1 -> 257.7 mm
- net +3V3: track 43.8 -> 45.2 mm
Changed lines of the file:
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@@
 (kicad_pcb (version 20160815) (host pcbnew "(2016-09-14 revision 83ed3c9)-makepkg")
   (general
-    (links 341)
-    (no_connects 10)
+    (links 343)
+    (no_connects 2)
     (area 42.949999 29.949999 120.550001 70.050001)
     (thickness 1.6)
     (drawings 158)
-    (tracks 1474)
+    (tracks 1478)
     (zones 0)
-    (modules 155)
+    (modules 157)
     (nets 115)
   )
@@
   )
   (module PCB_Footprints:TEST_POINT (layer F.Cu)
+    (at 51.025 68.375)
+    (fp_text reference TP35 (at 1.375 0.975) (layer F.SilkS)
+      (effects (font (size 0.5 0.5) (thickness 0.1)))
+    )
+    (fp_text value TEST_POINT (at 0.635 -2.413) (layer F.Fab)
+      (effects (font (size 0.5 0.5) (thickness 0.1)))
+    )
+    (pad 1 smd circle (at 0 0) (size 1.27 1.27) (layers F.Cu F.Paste F.Mask)
+      (net 2 GND) (solder_mask_margin 0.102))
+  )
+  (module PCB_Footprints:TEST_POINT (layer F.Cu)
+    (at 54.85 68.525)
+    (fp_text reference TP36 (at 0.05 1.1) (layer F.SilkS)
+      (effects (font (size 0.5 0.5) (thickness 0.1)))
+    )
+    (fp_text value TEST_POINT (at 0.635 -2.413) (layer F.Fab)
+      (effects (font (size 0.5 0.5) (thickness 0.1)))
+    )
+    (pad 1 smd circle (at 0 0) (size 1.27 1.27) (layers F.Cu F.Paste F.Mask)
+      (net 1 +3V3) (solder_mask_margin 0.102))
+  )
+  (module PCB_Footprints:TEST_POINT (layer F.Cu)
     (at 56.025 50.8)
-    (fp_text reference TP31 (at -0.075 -1.7 90) (layer F.SilkS)
+    (fp_text reference TP31 (at -0.375 -1.175 180) (layer F.SilkS)
       (effects (font (size 0.5 0.5) (thickness 0.1)))
     )
@@
   (module PCB_Footprints:TEST_POINT (layer F.Cu)
     (at 59.175 51.925)
-    (fp_text reference TP32 (at 0.075 -1.65 90) (layer F.SilkS)
+    (fp_text reference TP32 (at 0 1.075 180) (layer F.SilkS)
       (effects (font (size 0.5 0.5) (thickness 0.1)))
     )
@@
   (module PCB_Footprints:TEST_POINT (layer F.Cu)
     (at 58.075 50.75)
-    (fp_text reference TP33 (at 0.15 -1.6 90) (layer F.SilkS)
+    (fp_text reference TP33 (at -0.05 -1.025 180) (layer F.SilkS)
       (effects (font (size 0.5 0.5) (thickness 0.1)))
     )
@@
   (module PCB_Footprints:TEST_POINT (layer F.Cu)
     (at 60.275 50.7)
-    (fp_text reference TP34 (at 0 -1.7 90) (layer F.SilkS)
+    (fp_text reference TP34 (at 0 -1.025 180) (layer F.SilkS)
       (effects (font (size 0.5 0.5) (thickness 0.1)))
     )
@@
   (module PCB_Footprints:TEST_POINT (layer F.Cu)
     (at 57.075 52.025)
-    (fp_text reference TP30 (at 0.025 -1.7 90) (layer F.SilkS)
+    (fp_text reference TP30 (at 0 1.075 180) (layer F.SilkS)
       (effects (font (size 0.5 0.5) (thickness 0.1)))
     )
@@
   (module PCB_Footprints:TEST_POINT (layer F.Cu)
     (at 85.85 41.65)
-    (fp_text reference TP12 (at 1.65 0.35) (layer F.SilkS)
+    (fp_text reference TP12 (at 0.1 1.125) (layer F.SilkS)
       (effects (font (size 0.5 0.5) (thickness 0.1)))
     )
@@
   )
   (module PCB_Footprints:FIDUCIAL (layer F.Cu)
-    (at 52.325 68.7)
-    (fp_text reference FD2 (at 1.725 0.55) (layer F.SilkS)
+    (at 57.275 68.675)
+    (fp_text reference FD2 (at 1.725 0.825) (layer F.SilkS)
       (effects (font (size 0.5 0.5) (thickness 0.1)))
     )
@@
     (pad 1 thru_hole rect (at 0 0 180) (size 2.032 1.7272) (drill 1.016) (layers *.Cu *.Mask F.SilkS)
       (net 2 GND))
-    (model Pin_Headers.3dshapes/Pin_Header_Straight_1x03.wrl
-      (at (xyz 0 -0.1 0))
-      (scale (xyz 1 1 1))
-      (rotate (xyz 0 0 90))
-    )
   )
   (module PCB_Footprints:LED0603 (layer F.Cu)
@@
   (gr_line (start 120.5 30) (end 43 30) (layer Edge.Cuts) (width 0.1))
   (gr_line (start 120.5 30) (end 120.5 70) (layer Edge.Cuts) (width 0.1))
+  (segment (start 54.864 67.1576) (end 54.864 68.511) (width 0.1778) (layer F.Cu) (net 1))
+  (segment (start 54.864 68.511) (end 54.85 68.525) (width 0.1778) (layer F.Cu) (net 1))
   (segment (start 84.3 51.658) (end 84.015026 51.658) (width 0.1778) (layer F.Cu) (net 1))
   (segment (start 84.015026 51.658) (end 83.432708 51.075682) (width 0.1778) (layer F.Cu) (net 1))
@@
   (segment (start 54.0004 66.8528) (end 54.356 66.4972) (width 0.1778) (layer F.Cu) (net 1))
   (via (at 54.356 66.4972) (size 0.635) (drill 0.3302) (layers F.Cu B.Cu) (net 1))
+  (segment (start 51.0286 66.8528) (end 51.0286 68.3714) (width 0.1778) (layer F.Cu) (net 2))
+  (segment (start 51.0286 68.3714) (end 51.025 68.375) (width 0.1778) (layer F.Cu) (net 2))
   (segment (start 57.017 60.303) (end 57.017 60.6028) (width 0.381) (layer F.Cu) (net 2))
   (segment (start 57.0424 62.206) (end 57.017 62.1806) (width 0.1778) (layer F.Cu) (net 2))
